File: evelinverter/pcb/evelinverter.kicad_pcb (KiCad board)
At the start: 4 copper layers, 30.5 x 20 mm, 62 parts, among them J1 IN+, J10 enc, J11 hall, J2 IN-, J3 swd, J4 U, J5 V, J6 W, J9 i2c, Q1 AON7418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

Commit message: started redoing evelinverter
Parts:
- removed C1, C15, C19, C20, C21: 100n, Capacitor_SMD:C_0402_1005Metric
- removed C12, C13, C14, C27: 100n, Capacitor_SMD:C_0603_1608Metric
- removed C16, C17, C18: 1u, Capacitor_SMD:C_1206_3216Metric
- removed C2: 1u, Capacitor_SMD:C_0402_1005Metric
- removed C22, C23: 10u, Capacitor_SMD:C_0603_1608Metric
- removed C24: 10u, Capacitor_SMD:C_1210_3225Metric
- removed C25: 100n, Capacitor_SMD:C_0805_2012Metric
- removed C26: 33n, Capacitor_SMD:C_0603_1608Metric
- removed C28: 47u, Capacitor_SMD:C_0805_2012Metric
- removed C3: 10u, Capacitor_SMD:C_0402_1005Metric
- removed C4, C5: 16p, Capacitor_SMD:C_0402_1005Metric
- removed J1: IN+, a22verter:SolderPad
- removed J10: enc, a22verter:MOLEX_5055670851
- removed J11: hall, a22verter:MOLEX_5055670651
- removed J2: IN-, a22verter:SolderPad
- removed J3: swd, a22verter:MOLEX_5055670651
- removed J4: U, a22verter:SolderPad
- removed J5: V, a22verter:SolderPad
- removed J6: W, a22verter:SolderPad
- removed J9: i2c, a22verter:MOLEX_5055670451
- removed L1: 6.8u, Inductor_SMD:L_Wuerth_MAPI-4030
- removed NT1: NetTie_2, NetTie:NetTie-2_SMD_Pad0.5mm
- removed Q1, Q2, Q3, Q4, Q5, Q6: AON7418, a22verter:DFN3.3x3.3-EP
- removed R1: 0, Resistor_SMD:R_0402_1005Metric
- removed R10, R8, R9: 1m, Resistor_SMD:R_0805_2012Metric
- removed R11, R12, R15: 10k, Resistor_SMD:R_0402_1005Metric
- removed R13: 22k, Resistor_SMD:R_0402_1005Metric
- removed R14: 140k, Resistor_SMD:R_0402_1005Metric
- removed R2, R3, R4, R5, R6, R7: 16, Resistor_SMD:R_0402_1005Metric
- removed U1: STM32G071CBU3, Package_DFN_QFN:QFN-48-1EP_7x7mm_P0.5mm_EP5.45x5.45mm
- removed U2: DRV8300DRGE, Package_DFN_QFN:VQFN-24-1EP_4x4mm_P0.5mm_EP2.45x2.45mm
- removed U3, U4, U5: INA186, Package_TO_SOT_SMD:SOT-363_SC-70-6
- removed U6: AP1117-33, Package_TO_SOT_SMD:SOT-89-3
- removed U7: TPS62933, a22verter:SOT-583
- removed Y1: RH100-8, Crystal:Crystal_SMD_3225-4Pin_3.2x2.5mm
Routing:
- net +3V3: track 73.3 -> 0.00 mm, vias 8 -> 0
- net +12V: track 30.9 -> 0.00 mm, vias 3 -> 0
- net GNDA: track 27.1 -> 0.00 mm, vias 2 -> 0
- net /mcu/adc1_in0: track 22.4 -> 0.00 mm, vias 2 -> 0
- net /mcu/adc1_in1: track 19.0 -> 0.00 mm, vias 2 -> 0
- net /mcu/nrst: track 18.6 -> 0.00 mm, vias 2 -> 0
- net /mcu/adc1_in2: track 16.4 -> 0.00 mm, vias 2 -> 0
- net /drive/sense_vref: track 14.1 -> 0.00 mm
- net /mcu/adc1_in3: track 11.7 -> 0.00 mm, vias 2 -> 0
- net Net-(C14-Pad1): track 11.0 -> 0.00 mm, vias 2 -> 0
- net /drive/w_sense_line: track 10.5 -> 0.00 mm, vias 3 -> 0
- net VBUS: track 10.2 -> 0.00 mm, vias 28 -> 0
- net Net-(R3-Pad1): track 9.90 -> 0.00 mm, vias 2 -> 0
- net /mcu/i2c1_sda: track 9.87 -> 0.00 mm, vias 1 -> 0
- net /drive/u_sense_line: track 9.74 -> 0.00 mm, vias 1 -> 0
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- removed copper zone on F.Cu, net /drive/u_sense_line
- removed copper zone on F.Cu, net /drive/u_sense_load
- removed copper zone on F.Cu, net /drive/v_sense_line
- removed copper zone on F.Cu, net /drive/v_sense_load
- removed copper zone on F.Cu, net /drive/w_sense_line
- removed copper zone on F.Cu, net /drive/w_sense_load
- removed copper zone on B.Cu, net GND
- removed copper zone on F.Cu, net GND
- removed copper zone on In1.Cu, net GND
- removed copper zone on In2.Cu, net GND
- removed copper zone on In1.Cu, net VBUS
Other:
- board outline removed
- board text removed: "+"
- board text removed: "-"
- board text removed: "30V"
- board text removed: "a22.r01"
- board text removed: "enc"
- board text removed: "evelynmau.de"
- board text removed: "hall"
- board text removed: "i2c"
- board text removed: "swd"
